File: Sensorbox_Schaltplan/SensorBox/SensorBox.kicad_sch (KiCad schematic)
At the start: 0 parts

Commit message: big change - hardware
folders changed, new proj. assigned
Other:
- removed sheet Luftdruck-Sensor
- removed sheet Luftfeuchtigkeit-Sensor
- removed sheet Ozon-Sensor
- removed sheet Temperatur-Sensor
Changed lines of the file:
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@@
 	(generator_version "8.0")
 	(paper "A4")
-	(sheet
-		(at 109.22 21.59)
-		(size 33.02 19.05)
-		(fields_autoplaced yes)
-		(stroke
-			(width 0.1524)
-			(type solid)
-		)
-		(fill
-			(color 0 0 0 0.0000)
-		)
-		(property "Sheetname" "Luftfeuchtigkeit-Sensor"
-			(at 109.22 20.8784 0)
-			(effects
-				(font
-					(size 1.27 1.27)
-				)
-				(justify left bottom)
-			)
-		)
-		(property "Sheetfile" "Luftfeuchtigkeit_Sensor.kicad_sch"
-			(at 109.22 41.2246 0)
-			(effects
-				(font
-					(size 1.27 1.27)
-				)
-				(justify left top)
-			)
-		)
-		(instances
-			(project "SensorBox"
-				(path "/7cbe8151-7294-42e6-9c4e-6ec8952d674f"
-					(page "5")
-				)
-			)
-		)
-	)
-	(sheet
-		(at 107.95 107.95)
-		(size 33.02 20.32)
-		(fields_autoplaced yes)
-		(stroke
-			(width 0.1524)
-			(type solid)
-		)
-		(fill
-			(color 0 0 0 0.0000)
-		)
-		(property "Sheetname" "Luftdruck-Sensor"
-			(at 107.95 107.2384 0)
-			(effects
-				(font
-					(size 1.27 1.27)
-				)
-				(justify left bottom)
-			)
-		)
-		(property "Sheetfile" "Luftdruck_Sensor.kicad_sch"
-			(at 107.95 128.8546 0)
-			(effects
-				(font
-					(size 1.27 1.27)
-				)
-				(justify left top)
-			)
-		)
-		(instances
-			(project "SensorBox"
-				(path "/7cbe8151-7294-42e6-9c4e-6ec8952d674f"
-					(page "3")
-				)
-			)
-		)
-	)
-	(sheet
-		(at 109.22 50.8)
-		(size 26.67 16.51)
-		(fields_autoplaced yes)
-		(stroke
-			(width 0.1524)
-			(type solid)
-		)
-		(fill
-			(color 0 0 0 0.0000)
-		)
-		(property "Sheetname" "Temperatur-Sensor"
-			(at 109.22 50.0884 0)
-			(show_name yes)
-			(effects
-				(font
-					(size 1.27 1.27)
-				)
-				(justify left bottom)
-			)
-		)
-		(property "Sheetfile" "Temp_Sensor.kicad_sch"
-			(at 109.22 67.8946 0)
-			(show_name yes)
-			(effects
-				(font
-					(size 1.27 1.27)
-				)
-				(justify left top)
-			)
-		)
-		(instances
-			(project "SensorBox"
-				(path "/7cbe8151-7294-42e6-9c4e-6ec8952d674f"
-					(page "2")
-				)
-			)
-		)
-	)
-	(sheet
-		(at 107.95 78.74)
-		(size 27.94 19.05)
-		(fields_autoplaced yes)
-		(stroke
-			(width 0.1524)
-			(type solid)
-		)
-		(fill
-			(color 0 0 0 0.0000)
-		)
-		(property "Sheetname" "Ozon-Sensor"
-			(at 107.95 78.0284 0)
-			(effects
-				(font
-					(size 1.27 1.27)
-				)
-				(justify left bottom)
-			)
-		)
-		(property "Sheetfile" "Ozon_Sensor.kicad_sch"
-			(at 107.95 98.3746 0)
-			(effects
-				(font
-					(size 1.27 1.27)
-				)
-				(justify left top)
-			)
-		)
-		(instances
-			(project "SensorBox"
-				(path "/7cbe8151-7294-42e6-9c4e-6ec8952d674f"
-					(page "4")
-				)
-			)
-		)
-	)
 	(sheet_instances
 		(path "/"
