File: Sensorbox_allgemein/Externer_Sensor/ExternerSensor/ExternerSensor.kicad_sch (KiCad schematic)
At the start: 4 parts

Commit message: Externer Sensor
aufgebaut
Parts:
- added C1: 0.1uF, Capacitor_SMD:C_0402_1005Metric_Pad0.74x0.62mm_HandSolder, symbol Device:C
- added C2: 10uF, Capacitor_SMD:C_0402_1005Metric_Pad0.74x0.62mm_HandSolder, symbol Device:C
- added R1: 240R, Resistor_SMD:R_0402_1005Metric, symbol Device:R
- added R2, R3, R4, R5: 390R, Resistor_SMD:R_0402_1005Metric, symbol Device:R
- added R6: 68R, Resistor_SMD:R_0402_1005Metric, symbol Device:R
- added R7: 500R, Resistor_SMD:R_0402_1005Metric, symbol Device:R
- added TH1: PT100, Resistor_THT:R_Axial_DIN0204_L3.6mm_D1.6mm_P5.08mm_Horizontal, symbol Sensor_Temperature:PT100
- added U1: AMS1117, Package_TO_SOT_SMD:SOT-223-3_TabPin2, symbol Regulator_Linear:AMS1117
- added U2: INA333xxDGK, Package_SO:VSSOP-8_3.0x3.0mm_P0.65mm, symbol Amplifier_Instrumentation:INA333xxDGK
- added U3: ADS1115IDGS, Package_SO:TSSOP-10_3x3mm_P0.5mm, symbol Analog_ADC:ADS1115IDGS
- added U4: LM334M, Package_SO:SOIC-8_3.9x4.9mm_P1.27mm, symbol Reference_Current:LM334M
- renumbered GND1 to GND, SCL1 to SCL, SDA/Signal1 to SDA/Signal, VCC1 to VCC
Connections:
- net SCL: now reaches SCL.1 (Pin_1)
- net SCL: now also U3.10 (SCL)
- net SDA: now reaches SDA/Signal.1 (Pin_1)
- net SDA: now also U3.9 (SDA)
- net VCC: now reaches VCC.1 (Pin_1)
- net VCC: now also C1.1, U1.3 (VI), U4.4
- net GND1: now reaches GND.1 (Pin_1)
- net GND1: now also C1.2, C2.2, R2.2, R5.2, R6.2, TH1.1, U2.4 (V-), U2.5 (Ref), U3.1 (ADDR), U3.3 (GND)
- new net: R6.1, U4.1
- new net: R3.1, R4.1, U4.2, U4.3, U4.6, U4.7
- new net: R1.1, R2.1, U1.1 (ADJ)
- new net: R7.1, U2.1 (Rg)
- new net: R7.2, U2.8 (Rg)
- new net 3V3: C2.1, R1.2, U1.2 (VO), U2.7 (V+), U3.8 (VDD)
- new net 6_AIN0: U2.6, U3.4 (AIN0)
- new net V0: R3.2, R5.1, U2.3 (+)
- new net VL: R4.2, TH1.2, U2.2 (-)
Other:
- note added: "ADS wandelt Analog Signal in Digitale Daten um"
- note added: "LM erzeugt konstanten Strom"
- note added: "Spannungsregler 7.4V - 3.3V"
- note added: "Verstärkt die Differenz Spannung [V0-VL] der Wheat Stone Brücke"
- note added: "Wheat Stone Brücke wandelt die Widerstandänderung des PT-100 in eine Spannungsdifferenz"
- moved on the sheet: GND, SCL, SDA/Signal, VCC
