File: Sensorbox_HW/SensorBox/SensorBox.kicad_sch (KiCad schematic)
At the start: 80 parts, among them U1 BME280, U11 PS1-O3-100, U12 DS3231M, U13 OPA197xD, U2 OPA197xD, U4 MC33063AD, U5 OPA197xD, U6 MAX31855EASA, U8 HPP845E131R5

Commit message: änderung schaltplan (Anordnung)
Other:
- note removed: "Wichtig fürs Layout: Der Sensor der am Schluss der Datenleitung hängt Pullup Widerstände hängen. Hier BME!!!"
- moved on the sheet: ADC1, BT1, C10, C14, C5, C8, C9, CO1, CO2, CO4, CR1220, CT1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

Commit message: PCB: BME PAD länger designed und Befestigungslöcher hinzugefügt
Parts:
- removed U1: BME280, BME280 (2):BME280, symbol Sensor:BME280
- added U3: BME280, Package_LGA:Bosch_LGA-8_2.5x2.5mm_P0.65mm_ClockwisePinNumbering, symbol Sensor:BME280
Connections:
- net GND1: now also U3.1 (GND), U3.5 (SDO), U3.7 (GND)
- net SCL_GPIO22: now also U3.4 (SCK)
- net SDA_GPIO21: now also U3.3 (SDI)
- net VDD_3V3: now also U3.2 (CSB), U3.6 (VDDIO), U3.8 (VDD)
Changed lines of the file:
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@@
 		)
 		(instances
-			(project ""
+			(project "SensorBox"
 				(path "/7cbe8151-7294-42e6-9c4e-6ec8952d674f"
 					(reference "S1")
@@
 	)
 	(symbol
+		(lib_id "Sensor:BME280")
+		(at 34.29 140.97 270)
+		(unit 1)
+		(exclude_from_sim no)
+		(in_bom yes)
+		(on_board yes)
+		(dnp no)
+		(fields_autoplaced yes)
+		(property "Reference" "U3"
+			(at 34.29 125.73 90)
+			(effects
+				(font
+					(size 1.27 1.27)
+				)
+			)
+		)
+		(property "Value" "BME280"
+			(at 34.29 128.27 90)
+			(effects
+				(font
+					(size 1.27 1.27)
+				)
+			)
+		)
+		(property "Footprint" "Package_LGA:Bosch_LGA-8_2.5x2.5mm_P0.65mm_ClockwisePinNumbering"
+			(at 22.86 179.07 0)
+			(effects
+				(font
+					(size 1.27 1.27)
+				)
+				(hide yes)
+			)
+		)
+		(property "Datasheet" "https://www.bosch-sensortec.com/media/boschsensortec/downloads/datasheets/bst-bme280-ds002.pdf"
+			(at 29.21 140.97 0)
+			(effects
+				(font
+					(size 1.27 1.27)
+				)
+				(hide yes)
+			)
+		)
+		(property "Description" "3-in-1 sensor, humidity, pressure, temperature, I2C and SPI interface, 1.71-3.6V, LGA-8"
+			(at 34.29 140.97 0)
+			(effects
+				(font
+					(size 1.27 1.27)
+				)
+				(hide yes)
+			)
+		)
+		(pin "6"
+		)
+		(pin "4"
+		)
+		(pin "3"
+		)
+		(pin "1"
+		)
+		(pin "5"
+		)
+		(pin "2"
+		)
+		(pin "8"
+		)
+		(pin "7"
+		)
+		(instances
+			(project "SensorBox"
+				(path "/7cbe8151-7294-42e6-9c4e-6ec8952d674f"
+					(reference "U3")
+					(unit 1)
+				)
+			)
+		)
+	)
+	(symbol
 		(lib_id "Connector:Conn_01x01_Socket")
 		(at 273.05 105.41 0)
@@
 		)
 		(instances
-			(project ""
+			(project "SensorBox"
 				(path "/7cbe8151-7294-42e6-9c4e-6ec8952d674f"
 					(reference "L1")
@@
 					(unit 1)
 				)
-			)
-		)
-	)
-	(symbol
-		(lib_id "Sensor:BME280")
-		(at 34.29 140.97 270)
-		(unit 1)
-		(exclude_from_sim no)
-		(in_bom yes)
-		(on_board yes)
-		(dnp no)
-		(fields_autoplaced yes)
-		(property "Reference" "U1"
-			(at 34.29 125.73 90)
-			(effects
-				(font
-					(size 1.27 1.27)
-				)
-			)
-		)
-		(property "Value" "BME280"
-			(at 34.29 128.27 90)
-			(effects
-				(font
-					(size 1.27 1.27)
-				)
-			)
-		)
-		(property "Footprint" "BME280 (2):BME280"
-			(at 22.86 179.07 0)
-			(effects
-				(font
-					(size 1.27 1.27)
-				)
-				(hide yes)
-			)
-		)
-		(property "Datasheet" "https://www.bosch-sensortec.com/media/boschsensortec/downloads/datasheets/bst-bme280-ds002.pdf"
-			(at 29.21 140.97 0)
-			(effects
-				(font
-					(size 1.27 1.27)
-				)
-				(hide yes)
-			)
-		)
-		(property "Description" "3-in-1 sensor, humidity, pressure, temperature, I2C and SPI interface, 1.71-3.6V, LGA-8"
-			(at 34.29 140.97 0)
-			(effects
-				(font
-					(size 1.27 1.27)
-				)
-				(hide yes)
-			)
-		)
-		(pin "6"
-		)
-		(pin "2"
-		)
-		(pin "7"
-		)
-		(pin "8"
-		)
-		(pin "1"
-		)
-		(pin "3"
-		)
-		(pin "4"
-		)
-		(pin "5"
-		)
-		(instances
-			(project "SensorBox"
-				(path "/7cbe8151-7294-42e6-9c4e-6ec8952d674f"
-					(reference "U1")
-					(unit 1)
-				)

Commit message: HW-PCB-Change
Die HW wurde angepasst --> Leiterbahnen wurden abgecheckt und geändert; PCB vom BME geändert; GND-Flächen angepasst
Parts:
- U3: footprint Package_LGA:Bosch_LGA-8_2.5x2.5mm_P0.65mm_ClockwisePinNumbering -> BME_CHANGED:Bosch_LGA-8_2.5x2.5mm_P0.65mm_ClockwisePinNumbering_ch
Changed lines of the file:
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@@
 			)
 		)
-		(property "Footprint" "Package_LGA:Bosch_LGA-8_2.5x2.5mm_P0.65mm_ClockwisePinNumbering"
+		(property "Footprint" "BME_CHANGED:Bosch_LGA-8_2.5x2.5mm_P0.65mm_ClockwisePinNumbering_ch"
 			(at 22.86 179.07 0)
 			(effects
