File: Sensorbox_HW/Versionen/V4_07_2_2025/SensorBox/SensorBox.kicad_sch (KiCad schematic)
At the start: 81 parts, among them U1 BME280, U11 PS1-O3-100, U12 DS3231M, U13 OPA197xD, U2 OPA197xD, U4 MC33063AD, U5 OPA197xD, U6 MAX31855EASA, U8 HPP845E131R5

Commit message: änderung schaltplan (Anordnung)
Other:
- note removed: "Wichtig fürs Layout: Der Sensor der am Schluss der Datenleitung hängt Pullup Widerstände hängen. Hier BME!!!"
- moved on the sheet: ADC1, C10, C5, C8, C9, CO4, CR1220, D2, D4, D5, D7, GND1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
